Commit message: Added and tested some new objects

File: data/assets/objects/cylinder/object.urdf (robot description, URDF)
Before this commit: robot cross, 1 links, 0 joints
Links:
- link baseLink: geometry collision cylinder length=0.05 radius=0.025; visual cylinder length=0.05 radius=0.025

File: data/assets/objects_NOT_WORKING/double_t/object.urdf (robot description, URDF)
Before this commit: robot cross, 1 links, 0 joints
Links:
- link baseLink: geometry collision box size=0.08 0.025 0.05; collision box size=0.08 0.025 0.05

File: data/assets/objects_NOT_WORKING/triangle/object.urdf (robot description, URDF)
Before this commit: robot cross, 1 links, 0 joints
Links:
- link baseLink: geometry collision mesh filename=package://path/to/your/triangle.obj scale=1 1 1; visual mesh filename=package://path/to/your/triangle.obj scale=1 1 1
