Commit message: adapted URDF for use with cylider, also added minimal push animation

File: data/assets/urdf/robot.urdf (robot description, URDF)
Before this commit: robot ur10e_cell, 42 links, 41 joints
Links:
- removed link left_inner_finger
- removed link left_inner_finger_pad
- removed link left_inner_knuckle
- removed link left_outer_finger
- removed link left_outer_knuckle
- removed link right_inner_finger
- removed link right_inner_finger_pad
- removed link right_inner_knuckle
- removed link right_outer_finger
- removed link right_outer_knuckle
- removed link robotiq_arg2f_base_link
- added link cylinder_link, mass 0.5; collision cylinder length=0.4 radius=0.01; visual cylinder length=0.4 radius=0.01
Joints:
- removed joint finger_joint
- removed joint left_inner_finger_joint
- removed joint left_inner_finger_pad_joint
- removed joint left_inner_knuckle_joint
- removed joint left_outer_finger_joint
- removed joint mount_to_gripper_joint
- removed joint right_inner_finger_joint
- removed joint right_inner_finger_pad_joint
- removed joint right_inner_knuckle_joint
- removed joint right_outer_finger_joint
- removed joint right_outer_knuckle_joint
- added joint mount_to_tool_joint: type fixed, parent realsense_mount_base_link, child cylinder_link, origin xyz=0 0 0.007 rpy=0 0 1.5707963267948966
- joint tcp_joint: origin xyz=0 0 0.22 rpy=0 0 0 -> xyz=0 0 0.2 rpy=0 0 0
