Commit message: Added urdf and config files for all designated ares, remove material_name from object urdfs

File: data/assets/areas/cross/object.urdf (robot description, URDF)
Before this commit: robot t, 1 links, 0 joints
Links:
- link baseLink: geometry visual box size=0.035 0.09 0.0005; visual box size=0.09 0.035 0.0005

File: data/assets/areas/cube/object.urdf (robot description, URDF)
Before this commit: robot cylinder, 1 links, 0 joints
Links:
- link baseLink: geometry visual box size=0.06 0.06 0.0005

File: data/assets/areas/cylinder/object.urdf (robot description, URDF)
Before this commit: robot cylinder, 1 links, 0 joints
Links:
- link baseLink: geometry visual cylinder length=0.0005 radius=0.03

File: data/assets/areas/double_t/object.urdf (robot description, URDF)
Before this commit: robot t, 1 links, 0 joints
Links:
- link baseLink: geometry visual box size=0.035 0.09 0.0005; visual box size=0.09 0.035 0.0005

File: data/assets/areas/t/object.urdf (robot description, URDF)
Before this commit: robot t, 1 links, 0 joints
Links:
- link baseLink: geometry visual box size=0.035 0.09 0.0005; visual box size=0.09 0.035 0.0005
