Commit message: Deleted mass of areas to prevent gravity effects like falling through the ground, changed overlapping logic

File: data/assets/areas/cross/area.urdf (robot description, URDF)
Before this commit: robot cross, 1 links, 0 joints
Links:
- link baseLink: mass 0.2 -> 0.0

File: data/assets/areas/cube/area.urdf (robot description, URDF)
Before this commit: robot cube, 1 links, 0 joints
Links:
- link baseLink: mass 0.2 -> 0.0

File: data/assets/areas/cylinder/area.urdf (robot description, URDF)
Before this commit: robot cylinder, 1 links, 0 joints
Links:
- link baseLink: mass 0.2 -> 0.0

File: data/assets/areas/double_t/area.urdf (robot description, URDF)
Before this commit: robot t, 1 links, 0 joints
Links:
- link baseLink: mass 0.2 -> 0.0

File: data/assets/areas/t/area.urdf (robot description, URDF)
Before this commit: robot t, 1 links, 0 joints
Links:
- link baseLink: mass 0.2 -> 0.0
