Commit message: Fixed overlapping problem between areas and objects, recalcualte min_dist for all objects and areas, made Doppel_T and T smaller to prevent problem that no valid pose could be find

File: data/assets/areas/double_t/area.urdf (robot description, URDF)
Before this commit: robot t, 1 links, 0 joints
Links:
- link baseLink: geometry visual box size=0.03 0.06 0.0005; visual box size=0.06 0.03 0.0005

File: data/assets/areas/t/area.urdf (robot description, URDF)
Before this commit: robot t, 1 links, 0 joints
Links:
- link baseLink: geometry visual box size=0.03 0.06 0.0005; visual box size=0.06 0.03 0.0005

File: data/assets/objects/double_t/object.urdf (robot description, URDF)
Before this commit: robot t, 1 links, 0 joints
Links:
- link baseLink: geometry collision box size=0.02 0.05 0.05; collision box size=0.05 0.02 0.05

File: data/assets/objects/t/object.urdf (robot description, URDF)
Before this commit: robot t, 1 links, 0 joints
Links:
- link baseLink: geometry collision box size=0.02 0.05 0.05; collision box size=0.05 0.02 0.05
