Commit message: Adapted URDFs, updated ToDo

File: data/assets/objects/cross/object.urdf (robot description, URDF)
Before this commit: robot cross, 1 links, 0 joints
Links:
- link baseLink: mass 0.2 -> 0.19

File: data/assets/objects/cube/object.urdf (robot description, URDF)
Before this commit: robot cube, 1 links, 0 joints
Links:
- link baseLink: mass 0.2 -> 0.119

File: data/assets/objects/cylinder/object.urdf (robot description, URDF)
Before this commit: robot cylinder, 1 links, 0 joints
Links:
- link baseLink: mass 0.2 -> 0.0932

File: data/assets/objects/t/object.urdf (robot description, URDF)
Before this commit: robot t, 1 links, 0 joints
Links:
- link baseLink: mass 0.2 -> 0.095
