Commit message: Made obejcts bigger to make the training easier

File: data/assets/areas/cube/area.urdf (robot description, URDF)
Before this commit: robot cube, 1 links, 0 joints
Links:
- link baseLink: geometry visual box size=0.2 0.2 0.0005

File: data/assets/areas/cylinder/area.urdf (robot description, URDF)
Before this commit: robot cylinder, 1 links, 0 joints
Links:
- link baseLink: geometry visual cylinder length=0.0005 radius=0.1

File: data/assets/objects/cube/object.urdf (robot description, URDF)
Before this commit: robot cube, 1 links, 0 joints
Links:
- link baseLink: geometry collision box size=0.15 0.15 0.05; visual box size=0.15 0.15 0.05

File: data/assets/objects/cylinder/object.urdf (robot description, URDF)
Before this commit: robot cylinder, 1 links, 0 joints
Links:
- link baseLink: geometry collision cylinder length=0.05 radius=0.075; visual cylinder length=0.05 radius=0.075

Commit message: Changed the size of cube and cylinder object and area back to original (smaller) size

File: data/assets/areas/cube/area.urdf (robot description, URDF)
Before this commit: robot cube, 1 links, 0 joints
Links:
- link baseLink: geometry visual box size=0.06 0.06 0.0005

File: data/assets/areas/cylinder/area.urdf (robot description, URDF)
Before this commit: robot cylinder, 1 links, 0 joints
Links:
- link baseLink: geometry visual cylinder length=0.0005 radius=0.03

File: data/assets/objects/cube/object.urdf (robot description, URDF)
Before this commit: robot cube, 1 links, 0 joints
Links:
- link baseLink: geometry collision box size=0.05 0.05 0.05; visual box size=0.05 0.05 0.05

File: data/assets/objects/cylinder/object.urdf (robot description, URDF)
Before this commit: robot cylinder, 1 links, 0 joints
Links:
- link baseLink: geometry collision cylinder length=0.05 radius=0.025; visual cylinder length=0.05 radius=0.025
